File: Kicad/Labsheet2/Labsheet2.kicad_sch (KiCad schematic)
At the start: 0 parts

Commit message: Update Labsheet2.kicad_sch
Other:
- added sheet ESP32 (ESP32.kicad_sch)
- added sheet LEDs (LEDs.kicad_sch)
Changed lines of the file:
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@@
 (kicad_sch (version 20220622) (generator eeschema)
   (paper "A4")
-  (symbol_instances)
+  (wire (pts (xy 114.3 59.944) (xy 124.46 59.944))
+    (stroke (width 0) (type default))
+  )
+  (wire (pts (xy 114.3 65.024) (xy 124.46 65.024))
+    (stroke (width 0) (type default))
+  )
+  (wire (pts (xy 114.3 62.484) (xy 124.46 62.484))
+    (stroke (width 0) (type default))
+  )
+  (wire (pts (xy 114.3 57.404) (xy 124.46 57.404))
+    (stroke (width 0) (type default))
+  )
+  (wire (pts (xy 114.3 54.864) (xy 124.46 54.864))
+    (stroke (width 0) (type default))
+  )
+  (wire (pts (xy 114.3 67.564) (xy 124.46 67.564))
+    (stroke (width 0) (type default))
+  )
+  (wire (pts (xy 114.3 72.644) (xy 124.46 72.644))
+    (stroke (width 0) (type default))
+  )
+  (wire (pts (xy 114.3 70.104) (xy 124.46 70.104))
+    (stroke (width 0) (type default))
+  )
+  (sheet (at 97.028 50.8) (size 17.272 25.4) (fields_autoplaced)
+    (stroke (width 0.1524) (type solid))
+    (fill (color 0 0 0 0.0000))
+    (property "Sheetname" "ESP32" (id 0) (at 97.028 50.0884 0)
+      (effects (font (size 1.27 1.27)) (justify left bottom))
+    )
+    (property "Sheetfile" "ESP32.kicad_sch" (id 1) (at 97.028 76.7846 0)
+      (effects (font (size 1.27 1.27)) (justify left top) hide)
+    )
+    (pin "GPIO.23" output (at 114.3 54.864 0)
+      (effects (font (size 1.27 1.27)) (justify right))
+    )
+    (pin "GPIO.01" output (at 114.3 59.944 0)
+      (effects (font (size 1.27 1.27)) (justify right))
+    )
+    (pin "GPIO.22" output (at 114.3 57.404 0)
+      (effects (font (size 1.27 1.27)) (justify right))
+    )
+    (pin "GPIO.18" output (at 114.3 70.104 0)
+      (effects (font (size 1.27 1.27)) (justify right))
+    )
+    (pin "GPIO.03" output (at 114.3 62.484 0)
+      (effects (font (size 1.27 1.27)) (justify right))
+    )
+    (pin "GPIO.19" output (at 114.3 67.564 0)
+      (effects (font (size 1.27 1.27)) (justify right))
+    )
+    (pin "GPIO.21" output (at 114.3 65.024 0)
+      (effects (font (size 1.27 1.27)) (justify right))
+    )
+    (pin "GPIO.05" output (at 114.3 72.644 0)
+      (effects (font (size 1.27 1.27)) (justify right))
+    )
+  )
+  (sheet (at 124.46 50.8) (size 12.7 25.4) (fields_autoplaced)
+    (stroke (width 0.1524) (type solid))
+    (fill (color 0 0 0 0.0000))
+    (property "Sheetname" "LEDs" (id 0) (at 124.46 50.0884 0)
+      (effects (font (size 1.27 1.27)) (justify left bottom))
+    )
+    (property "Sheetfile" "LEDs.kicad_sch" (id 1) (at 124.46 77.0386 0)
+      (effects (font (size 1.27 1.27)) (justify left top) hide)
+    )
+    (pin "LED.1" input (at 124.46 54.864 180)
+      (effects (font (size 1.27 1.27)) (justify left))
+    )
+    (pin "LED.2" input (at 124.46 57.404 180)
+      (effects (font (size 1.27 1.27)) (justify left))
+    )
+    (pin "LED.3" input (at 124.46 59.944 180)
+      (effects (font (size 1.27 1.27)) (justify left))
+    )
+    (pin "LED.4" input (at 124.46 62.484 180)
+      (effects (font (size 1.27 1.27)) (justify left))
+    )
+    (pin "LED.5" input (at 124.46 65.024 180)
+      (effects (font (size 1.27 1.27)) (justify left))
+    )
+    (pin "LED.6" input (at 124.46 67.564 180)
+      (effects (font (size 1.27 1.27)) (justify left))
+    )
+    (pin "LED.7" input (at 124.46 70.104 180)
+      (effects (font (size 1.27 1.27)) (justify left))
+    )
+    (pin "LED.8" input (at 124.46 72.644 180)
+      (effects (font (size 1.27 1.27)) (justify left))
+    )
+  )
+  (sheet_instances
+    (path "/" (page "1"))
+    (path "/6b627919-67ca-436f-9087-d11f2bdbecf6" (page "2"))
+    (path "/b85758e4-c2e8-4c8e-9b7a-d843238d2e89" (page "3"))
+  )
 )
